File: dmx2uart.brd (EAGLE design)
At the start: 19.4 x 41.3 mm, 6 parts, among them IC1 MAX487

Commit message: capacitor size
Parts:
- C1: value 100uF -> 100nF
Changed lines of the file:
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@@
 <layer number="21" name="tPlace" color="7" fill="1" visible="yes" active="yes"/>
 <layer number="22" name="bPlace" color="7" fill="1" visible="yes" active="yes"/>
-<layer number="23" name="tOrigins" color="15" fill="1" visible="yes" active="yes"/>
-<layer number="24" name="bOrigins" color="15" fill="1" visible="yes" active="yes"/>
+<layer number="23" name="tOrigins" color="15" fill="1" visible="no" active="yes"/>
+<layer number="24" name="bOrigins" color="15" fill="1" visible="no" active="yes"/>
 <layer number="25" name="tNames" color="7" fill="1" visible="yes" active="yes"/>
 <layer number="26" name="bNames" color="7" fill="1" visible="yes" active="yes"/>
@@
 <attribute name="OC_FARNELL" value="unknown" x="49.53" y="19.05" size="1.778" layer="27" display="off"/>
 </element>
-<element name="C1" library="rcl" package="C075-032X103" value="100uF" x="29.21" y="34.29" smashed="yes">
+<element name="C1" library="rcl" package="C075-032X103" value="100nF" x="29.21" y="34.29" smashed="yes">
 <attribute name="VALUE" x="34.544" y="33.782" size="1.27" layer="27" ratio="10"/>
 </element>
